Commit message: Removed problematic floating_base_joint

File: urdf/g1/g1_23dof.urdf (robot description, URDF)
Before this commit: robot g1_23dof, 37 links, 36 joints
Links:
- removed link world
Joints:
- removed joint floating_base_joint

File: urdf/g1/ros2_control_23dof.xacro (robot description, xacro)
@@ -33,8 +33,8 @@
         </sensor>
         <!-- ADD THIS FLOATING BASE JOINT -->
-        <joint name="floating_base_joint">
+        <!-- <joint name="floating_base_joint">
             <state_interface name="position"/>
             <state_interface name="velocity"/>
-        </joint>
+        </joint> -->
         <xacro:joint_interface name="left_hip_pitch_joint" initial_pos="-0.1"/>
         <xacro:joint_interface name="left_hip_roll_joint" initial_pos="0"/>
